File: E-MATCH.kicad_sch (KiCad schematic)
At the start: 7 parts, among them IC1 NCV81071BZR2G, J2 691137710002, Q2 AOSP36326C, U1 TMCS1108A2UQDR

Commit message: linked 3-d models
Parts:
- removed J2: 691137710002, Screw_Terminal_0102:691137710002, symbol Screw Terminal:691137710002
- added J1: 691210910002, Screw_Terminal:691210910002, symbol Screw Terminal:691210910002
Connections:
- net at CR1.1, U1.3 (IN-), U1.4 (IN-): now also J1.2
- net at CR1.2, Q2.5, Q2.6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: now also J1.1
Changed lines of the file:
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@@
-	)
-	(symbol
-		(lib_id "Screw Terminal:691137710002")
-		(at 41.91 92.71 90)
-		(unit 1)
-		(exclude_from_sim no)
-		(in_bom yes)
-		(on_board yes)
-		(dnp no)
-		(fields_autoplaced yes)
-		(property "Reference" "J2"
-			(at 43.18 86.36 90)
-			(effects
-				(font
-					(size 1.27 1.27)
-				)
-			)
-		)
-		(property "Value" "691137710002"
-			(at 43.18 88.9 90)
-			(effects
-				(font
-					(size 1.27 1.27)
-				)
-			)
-		)
-		(property "Footprint" "Screw_Terminal_0102:691137710002"
-			(at 41.91 92.71 0)
-			(effects
-				(font
-					(size 1.27 1.27)
-				)
-				(justify bottom)
-				(hide yes)
-			)
-		)
-		(property "Datasheet" ""
-			(at 41.91 92.71 0)
-			(effects
-				(font
-					(size 1.27 1.27)
-				)
-				(hide yes)
-			)
-		)
-		(property "Description" ""
-			(at 41.91 92.71 0)
-			(effects
-				(font
-					(size 1.27 1.27)
-				)
-				(hide yes)
-			)
-		)
-		(property "DigiKey_Part_Number" "732-10955-ND"
-			(at 41.91 92.71 0)
-			(effects
-				(font
-					(size 1.27 1.27)
-				)
-				(justify bottom)
-				(hide yes)
-			)
-		)
-		(property "SnapEDA_Link" "https://www.snapeda.com/parts/691137710002/W%25C3%25BCrth+Elektronik+Midcom/view-part/?ref=snap"
-			(at 41.91 92.71 0)
-			(effects
-				(font
-					(size 1.27 1.27)
-				)
-				(justify bottom)
-				(hide yes)
-			)
-		)
-		(property "Description_1" "2 Position Wire to Board Terminal Block Horizontal with Board 0.197 (5.00mm) Through Hole"
-			(at 41.91 92.71 0)
-			(effects
-				(font
-					(size 1.27 1.27)
-				)
-				(justify bottom)
-				(hide yes)
-			)
-		)
-		(property "MF" "Würth Elektronik"
-			(at 41.91 92.71 0)
-			(effects
-				(font
-					(size 1.27 1.27)
-				)
-				(justify bottom)
-				(hide yes)
-			)
-		)
-		(property "Package" "None"
-			(at 41.91 92.71 0)
-			(effects
-				(font
-					(size 1.27 1.27)
-				)
-				(justify bottom)
-				(hide yes)
-			)
-		)
-		(property "Check_prices" "https://www.snapeda.com/parts/691137710002/W%25C3%25BCrth+Elektronik+Midcom/view-part/?ref=eda"
-			(at 41.91 92.71 0)
-			(effects
-				(font
-					(size 1.27 1.27)
-				)
-				(justify bottom)
-				(hide yes)
-			)
-		)
-		(property "MP" "691137710002"
-			(at 41.91 92.71 0)
-			(effects
-				(font
-					(size 1.27 1.27)
-				)
-				(justify bottom)
-				(hide yes)
-			)
-		)
-		(pin "2"
-		)
-		(pin "1"
-		)
-		(instances
-			(project ""
-				(path "/ac49d8b8-9946-4b6b-9646-a2b20606c52a"
-					(reference "J2")
-					(unit 1)
-				)
-			)
-		)
 	)
 	(symbol
@@
 					(unit 1)
 				)
+			)
+		)
+	)
+	(symbol
+		(lib_id "Screw Terminal:691210910002")
+		(at 41.91 92.71 90)
+		(unit 1)
+		(exclude_from_sim no)
+		(in_bom yes)
+		(on_board yes)
+		(dnp no)
+		(fields_autoplaced yes)
+		(property "Reference" "J1"
+			(at 43.18 86.36 90)
+			(effects
+				(font
+					(size 1.27 1.27)
+				)
+			)
+		)
+		(property "Value" "691210910002"
+			(at 43.18 88.9 90)
+			(effects
+				(font
+					(size 1.27 1.27)
+				)
+			)
+		)
+		(property "Footprint" "Screw_Terminal:691210910002"
+			(at 41.91 92.71 0)
+			(effects
+				(font
+					(size 1.27 1.27)
+				)
+				(justify bottom)
+				(hide yes)
+			)
+		)
+		(property "Datasheet" ""
+			(at 41.91 92.71 0)
+			(effects
+				(font
+					(size 1.27 1.27)
+				)
+				(hide yes)
+			)
+		)
+		(property "Description" ""
+			(at 41.91 92.71 0)
+			(effects
+				(font
+					(size 1.27 1.27)
+				)
+				(hide yes)
+			)
+		)
+		(property "DigiKey_Part_Number" "732-691210910002-ND"
+			(at 41.91 92.71 0)
+			(effects
+				(font
+					(size 1.27 1.27)
+				)
+				(justify bottom)
+				(hide yes)
+			)
+		)
+		(property "SnapEDA_Link" "https://www.snapeda.com/parts/691210910002/W%25C3%25BCrth+Elektronik+Midcom/view-part/?ref=snap"
+			(at 41.91 92.71 0)
+			(effects
+				(font
+					(size 1.27 1.27)
+				)
+				(justify bottom)
+				(hide yes)
+			)
+		)
+		(property "Description_1" "2 Position Wire to Board Terminal Block Horizontal with Board 0.100 (2.54mm) Through Hole"
+			(at 41.91 92.71 0)
+			(effects
+				(font
+					(size 1.27 1.27)
+				)
+				(justify bottom)
+				(hide yes)
+			)
+		)
+		(property "MF" "Würth Elektronik"
+			(at 41.91 92.71 0)
+			(effects
+				(font
+					(size 1.27 1.27)
+				)
+				(justify bottom)
+				(hide yes)
+			)
+		)
+		(property "Package" "None"
+			(at 41.91 92.71 0)
+			(effects
+				(font
+					(size 1.27 1.27)
+				)
+				(justify bottom)
+				(hide yes)
+			)
+		)
+		(property "Check_prices" "https://www.snapeda.com/parts/691210910002/W%25C3%25BCrth+Elektronik+Midcom/view-part/?ref=eda"
+			(at 41.91 92.71 0)
+			(effects
+				(font
+					(size 1.27 1.27)
+				)
+				(justify bottom)
+				(hide yes)
+			)
+		)
+		(property "MP" "691210910002"
+			(at 41.91 92.71 0)
+			(effects
+				(font
+					(size 1.27 1.27)
+				)
+				(justify bottom)
+				(hide yes)
+			)
+		)
+		(pin "2"
+		)
+		(pin "1"
+		)
+		(instances
+			(project ""
+				(path "/ac49d8b8-9946-4b6b-9646-a2b20606c52a"
+					(reference "J1")
+					(unit 1)
+				)

Commit message: A lot of changes :)
Parts:
- added CR2, CR3, CR4: MSS1P5-M3/89A, DIODE_MSP3V3, symbol Schottcky Diode:MSS1P5-M3_89A
- added IC2: NCV81071BZR2G, Gate Driver:SOP65P490X110-9N, symbol Gate Driver:NCV81071BZR2G
- added J2, J3, J4: 691210910002, Screw_Terminal:691210910002, symbol Screw Terminal:691210910002
- added Q2, Q3, Q4: AOSP36326C, SO8SOP-8L_AOS, symbol N-Ch Mosfet:AOSP36326C
- added R2, R3, R4: 10R, Gate Resistor:RES_RC1206_YAG, symbol Device:R
- IC1: footprint Current Sensor:D0008A-IPC_A -> Gate Driver:SOP65P490X110-9N
- R1: value R -> 10R
- U1: footprint Gate Driver:SOP65P490X110-9N -> Current Sensor:D0008A-MFG
- renumbered Q2 to Q1
Connections:
- net Enable_Signal: now also IC2.1 (ENA)
- net GND: now also IC2.3 (ENB), IC2.4 (INB), IC2.5 (GND), Q2.1, Q2.2, Q2.3, Q3.1, Q3.2, Q3.3, Q4.1, Q4.2, Q4.3
- net Trigger_Signal: now also IC2.2 (INA)
- net VBAT: now also IC2.8 (VDD)
- net at CR1.1, J1.2, U1.3 (IN-)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: now also CR2.1, CR3.1, CR4.1, J2.2, J3.2, J4.2
- net Gate_Drive2: now reaches IC1.6 (OUTB)
- net at R1.2: no longer IC1.7 (OUTA)
- new net: CR2.2, J2.1, Q2.5, Q2.6, Q2.7, Q2.8
- new net: CR4.2, J4.1, Q4.5, Q4.6, Q4.7, Q4.8
- new net: Q3.4, R3.1
- new net: CR3.2, J3.1, Q3.5, Q3.6, Q3.7, Q3.8
- new net: Q4.4, R4.1
- new net: Q2.4, R2.1
- new net Gate_Drive1: IC1.7 (OUTA)
- new net Gate_Drive3: IC2.7 (OUTA)
- new net Gate_Drive4: IC2.6 (OUTB)
- no-connect marks 0 -> 1
Other:
- note removed: "Mosfet Gate"
- moved on the sheet: A1, CR1, IC1
