File: E-MATCH.kicad_pcb (KiCad board)
At the start: 4 copper layers, 100 x 100 mm, 32 parts, among them IC1 NCV81071BZR2G, IC2 NCV81071BZR2G, J1 691210910002, J2 691210910002, J3 691210910002, J4 691210910002, J5 DC Jack, M1 FDC8878, Q1 AOSP36326C, Q2 AOSP36326C, Q3 AOSP36326C, Q4 AOSP36326C, Q5 FDD1600N10ALZ, U1 TMCS1108A2UQDR

Commit message: added a trace
Routing:
- net Net-(CR1-Pad1): track 0.00 -> 17.1 mm

Commit message: added a copper pour
Routing:
- added copper zone on F.Cu, net GND
Changed lines of the file:
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@@
 		(net "Net-(CR1-Pad1)")
+	)
+	(zone
+		(net "GND")
+		(layer "F.Cu")
+		(hatch edge 0.5)
+		(connect_pads
+			(clearance 0.5)
+		)
+		(min_thickness 0.25)
+		(fill yes
+			(thermal_gap 0.5)
+			(thermal_bridge_width 0.5)
+			(island_removal_mode 0)
+		)
+		(polygon
+			(pts
+				(xy 92.6 38.4) (xy 205.6 38.4) (xy 205.6 149.6) (xy 92.6 149.6)
+			)
+		)
 	)
 	(embedded_fonts no)
